File: din_power_atm90e26.sch (KiCad schematic (older format))
At the start: 62 parts, among them J1 CONN_01X06, J2 VBAT, J3 CONN_01X08, J4 CONN_02X18, J5 CONN_01X08, U1 MCP73831-2-OT, U2 AP7365-33YG-13, U3 AP7365-33YG-13, U4 Hi-Link_SMPS, U5 dc-dc

Commit message: updated readme.
Parts:
- removed C4, C5, C6, C7, C8, C9: 1uF, Capacitors_SMD:C_0603, symbol device:C
- removed D1: D_Schottky, Diodes_SMD:D_SOD-323F, symbol device:D_Schottky
- removed D2: LED, LEDs:LED_0603, symbol device:LED
- removed J2: VBAT, Connectors_JST:JST_SH_BM02B-SRSS-TB_02x1.00mm_Straight, symbol din_power_atm90e26-rescue:CONN_01X02
- removed J3, J5: CONN_01X08, Connectors_Molex:Molex_NanoFit_2x04x2.50mm_Angled, symbol din_power_atm90e26-rescue:CONN_01X08
- removed J4: CONN_02X18, hi-link_smps:PCIE-36-SKT, symbol din_power_atm90e26-rescue:CONN_02X18
- removed R10, R11, R18, R19, R20, R21, R28, R29, R3, R30, R31, R4: 5.8R, Resistors_SMD:R_0603, symbol device:R
- removed R32: 2K, Resistors_SMD:R_0603, symbol device:R
- removed R33: 1K, Resistors_SMD:R_0603, symbol device:R
- removed U1: MCP73831-2-OT, TO_SOT_Packages_SMD:SOT-23-5, symbol din_power_atm90e26-rescue:MCP73831-2-OT
- removed U2, U3: AP7365-33YG-13, TO_SOT_Packages_SMD:SOT-89-3, symbol din_power_atm90e26-rescue:AP7365-33YG-13
- added J2: Conn_02x06_Counter_Clockwise, symbol conn:Conn_02x06_Counter_Clockwise
- added J3, J4: Conn_01x02, symbol conn:Conn_01x02
- R1, R2, R8, R9: footprint Resistors_SMD:R_0603 -> Resistor_SMD:R_0603_1608Metric
- R25, R26, R27: footprint Resistors_SMD:R_0603 -> Resistor_SMD:R_0805_2012Metric; PN R0603 -> R
- U4: PN HKLPM01 -> HLK-PM03
- U5: PN ROE-0505S -> RNM-3.33.3S
Connections:
- net +5V is gone; now on net +3V3: U4.4 (+VO), U5.2 (IN+)
- net +5V_ISO is gone; now on net +3.3V_ISO: U5.4 (OUT+)
- net +3.3V_ISO: now also J2.11 (Pin_11)
- net +3V3: now also J2.12 (Pin_12)
- net GNDA: now also J2.6 (Pin_6)
- net GNDPWR: now also J2.5 (Pin_5)
- net IA1+: now also J2.1 (Pin_1), J3.1 (Pin_1)
- net IA1-: now also J2.2 (Pin_2), J3.2 (Pin_2)
- net IB1+: now also J2.3 (Pin_3), J4.1 (Pin_1)
- net IB1-: now also J2.4 (Pin_4), J4.2 (Pin_2)
- net UA_SAMP: now also J2.7 (Pin_7)
- net UB_SAMP: now also J2.8 (Pin_8)
- net UC_SAMP: now also J2.9 (Pin_9)
Other:
- note removed: "Option N-CT2"
- note removed: "Optional N-CT1"
- note removed: "Power Systems - Battery and 3.3V"
- moved on the sheet: R8, R9

Commit message: added image and updated readme
Parts:
- removed J2: Conn_02x06_Counter_Clockwise, symbol conn:Conn_02x06_Counter_Clockwise
- removed J3, J4: Conn_01x02, symbol conn:Conn_01x02
- removed R8, R9: 5.8R, Resistor_SMD:R_0603_1608Metric, symbol device:R
- added C4: 1u, Resistor_SMD:R_0805_2012Metric, symbol device:C
- added D?: IND_LED, symbol device:LED
- added J2: Conn_02x18_Counter_Clockwise, hi-link_smps:PCIE-36-SKT, symbol conn:Conn_02x18_Counter_Clockwise
- added J? (x2): Audio-Jack-3, symbol conn:Audio-Jack-3
- added R? (x2): 5.8R, Resistor_SMD:R_0603_1608Metric, symbol device:R
- added R?: 499, symbol device:R
Connections:
- net +3.3V_ISO: now also J2.2 (Pin_2)
- net +3V3: now also C4.1, D?.2 (A), J2.1 (Pin_1)
- net GNDA: now also J2.18 (Pin_18), R?.1, R?.2
- net GNDPWR: now also C4.2, J2.17 (Pin_17), R?.2
- net IA1+: now also J2.22 (Pin_22), J?.1
- net IA1-: now also J2.21 (Pin_21), J?.3
- net IB1+: now also J2.20 (Pin_20), J?.1, R?.2
- net IB1-: now also J2.19 (Pin_19), J?.3, R?.1
- net UA_SAMP: now also J2.36 (Pin_36)
- net UB_SAMP: now also J2.35 (Pin_35)
- net UC_SAMP: now also J2.34 (Pin_34)
- new net: D?.1 (K), R?.1
Other:
- note added: "Connector for Metering/Processor boards."
- note added: "Power System"
- note removed: "Connector for Metering/Processor boards - Supplies IV samples \nand +5V power with/without isolation"
- note removed: "Power Systems (5V)"
- moved on the sheet: R1, R2
