File: _saved_din_power_atm90e26.sch (KiCad schematic (older format))
At the start: 46 parts, among them J1 CONN_01X06, J2 Conn_02x18_Counter_Clockwise, U1 TRS35_3, U2 TRS35_3, U3 AP7365-33YG-13, U4 Hi-Link_SMPS, U5 dc-dc, U6 AP7365-33YG-13

Commit message: minor updates.
Connections:
- net UC: no longer U4.1 (AC_L)
- net +3.3V_ISO renamed 3V3_METER
- net UA_SAMP renamed VP_0
- net UB_SAMP renamed VP_1
- net UC_SAMP renamed V_ACDC
- net V_ACDC: now also U4.1 (AC_L); no longer J2.34 (Pin_34)
Changed lines of the file:
@@
 UA
 Text GLabel 4800 2500 0    60   Input ~ 0
-UC
+V_ACDC
 Text GLabel 4800 2800 0    60   Input ~ 0
 UN
@@
 $EndComp
 Text GLabel 3350 1050 2    60   Input ~ 0
-UA_SAMP
+VP_0
 Text GLabel 3300 2050 2    60   Input ~ 0
-UB_SAMP
+VP_1
 Text GLabel 3300 2850 2    60   Input ~ 0
-UC_SAMP
+V_ACDC
 Text GLabel 9000 3850 2    60   Input ~ 0
-UA_SAMP
+VP_0
 Text GLabel 9000 3950 2    60   Input ~ 0
-UB_SAMP
-Text GLabel 9000 4050 2    60   Input ~ 0
-UC_SAMP
+VP_1
 Text GLabel 8500 5550 0    60   Input ~ 0
-GNDA
+GND_METER
 Text GLabel 8500 3950 0    60   Input ~ 0
-+3.3V_ISO
+3V3_METER
 Text GLabel 8500 5450 0    60   Input ~ 0
-GNDPWR
+GND_CPU
 Text GLabel 8500 3850 0    60   Input ~ 0
-+3V3
+3V3_CPU
 Text Label 5200 2800 3    60   ~ 0
 UN_IN
@@
 Text GLabel 6200 2250 2    60   Input ~ 0
 +5V
-Text GLabel 5000 1550 3    60   Input ~ 0
-GNDA
 $Comp
 L whatnick:LOGO G1
@@
 Connection ~ 5600 4100
 Text GLabel 6450 4100 2    60   Input ~ 0
-+3.3V_ISO
+3V3_METER
 $Comp
 L din_power_atm90e26-rescue:AP7365-33YG-13 U6
@@
 Connection ~ 5600 5400
 Text GLabel 6600 5400 3    60   Input ~ 0
-+3V3
+3V3_CPU
 $Comp
 L power:+5V #PWR0105
@@
 Text GLabel 9000 5550 2    60   Input ~ 0
 I1N_1_IN
+Text GLabel 4900 4650 3    60   Input ~ 0
+GND_METER
+Text GLabel 4950 5950 3    60   Input ~ 0
+GND_CPU
 $EndSCHEMATC
