File: _saved_din_power_atm90e26.sch (KiCad schematic (older format))
At the start: 39 parts, among them J1 CONN_01X06, J2 PCI_Express, U1 TRS35_3, U2 TRS35_3, U3 AP7365-33YG-13, U4 Hi-Link_SMPS, U5 dc-dc, U6 AP7365-33YG-13

Commit message: updated readme
Parts:
- R3, R4: value 5.8R -> 5.8; Spice_Model (none) -> 5.8; Spice_Netlist_Enabled (none) -> Y; Spice_Primitive (none) -> R
Connections:
- no-connect marks 28 -> 30
Changed lines of the file:
@@
 L graphic_symbols:SYM_Flash_Small SYM1
 U 1 1 59F73620
-P 8250 2600
-F 0 "SYM1" V 8160 2600 50  0001 C CNN
-F 1 "SYM_Flash_Small" V 8340 2600 50  0001 C CNN
-F 2 "Whatnick_logo:Fsilk_HV" H 8250 2575 50  0001 C CNN
-F 3 "" H 8650 2500 50  0001 C CNN
-F 4 "X" H 8250 2600 50  0001 C CNN "PN"
-F 5 "1" V 8250 2600 60  0001 C CNN "DNP"
-	1    8250 2600
+P 8400 1600
+F 0 "SYM1" V 8310 1600 50  0001 C CNN
+F 1 "SYM_Flash_Small" V 8490 1600 50  0001 C CNN
+F 2 "Whatnick_logo:Fsilk_HV" H 8400 1575 50  0001 C CNN
+F 3 "" H 8800 1500 50  0001 C CNN
+F 4 "X" H 8400 1600 50  0001 C CNN "PN"
+F 5 "1" V 8400 1600 60  0001 C CNN "DNP"
+	1    8400 1600
 	1    0    0    -1
 $EndComp
@@
 L whatnick:LOGO G1
 U 1 1 59F74376
-P 9000 2600
-F 0 "G1" H 9000 2498 60  0001 C CNN
-F 1 "LOGO" H 9000 2702 60  0001 C CNN
-F 2 "Whatnick_logo:Whatnick_logo" H 9000 2600 60  0001 C CNN
-F 3 "" H 9000 2600 60  0001 C CNN
-F 4 "X" H 9000 2600 50  0001 C CNN "PN"
-F 5 "1" H 9000 2600 60  0001 C CNN "DNP"
-	1    9000 2600
+P 9550 1550
+F 0 "G1" H 9550 1448 60  0001 C CNN
+F 1 "LOGO" H 9550 1652 60  0001 C CNN
+F 2 "Whatnick_logo:Whatnick_logo" H 9550 1550 60  0001 C CNN
+F 3 "" H 9550 1550 60  0001 C CNN
+F 4 "X" H 9550 1550 50  0001 C CNN "PN"
+F 5 "1" H 9550 1550 60  0001 C CNN "DNP"
+	1    9550 1550
 	1    0    0    -1
 $EndComp
@@
 P 2600 5900
 F 0 "R3" V 2393 5900 50  0000 C CNN
-F 1 "5.8R" V 2484 5900 50  0000 C CNN
+F 1 "5.8" V 2484 5900 50  0000 C CNN
 F 2 "Resistor_SMD:R_0603_1608Metric" V 2530 5900 50  0001 C CNN
 F 3 "" H 2600 5900 50  0001 C CNN
 F 4 "R0603" H 2600 5900 50  0001 C CNN "PN"
 F 5 "CPF0603B5R76E1" H 2600 5900 60  0001 C CNN "manf#"
+F 6 "R" H 2600 5900 50  0001 C CNN "Spice_Primitive"
+F 7 "5.8" H 2600 5900 50  0001 C CNN "Spice_Model"
+F 8 "Y" H 2600 5900 50  0001 C CNN "Spice_Netlist_Enabled"
 	1    2600 5900
 	-1   0    0    1
@@
 P 2600 6300
 F 0 "R4" V 2393 6300 50  0000 C CNN
-F 1 "5.8R" V 2484 6300 50  0000 C CNN
+F 1 "5.8" V 2484 6300 50  0000 C CNN
 F 2 "Resistor_SMD:R_0603_1608Metric" V 2530 6300 50  0001 C CNN
 F 3 "" H 2600 6300 50  0001 C CNN
 F 4 "R0603" H 2600 6300 50  0001 C CNN "PN"
+F 5 "R" H 2600 6300 50  0001 C CNN "Spice_Primitive"
+F 6 "5.8" H 2600 6300 50  0001 C CNN "Spice_Model"
+F 7 "Y" H 2600 6300 50  0001 C CNN "Spice_Netlist_Enabled"
 	1    2600 6300
 	-1   0    0    1
@@
 Text GLabel 8300 4700 0    60   Input ~ 0
 I1N_0_N
+Text GLabel 8300 3900 0    60   Input ~ 0
+I1P_1_IN
 Text GLabel 8300 3500 0    60   Input ~ 0
-I1P_1_IN
-Text GLabel 8300 3300 0    60   Input ~ 0
 I1N_1_IN
 Text GLabel 4950 4900 3    60   Input ~ 0
@@
 NoConn ~ 8500 3700
 NoConn ~ 8500 3800
-NoConn ~ 8500 3900
 NoConn ~ 8500 4000
 NoConn ~ 8500 4100
@@
 	750  7050 3750 7050
 Wire Notes Line
-	9500 3000 9500 5900
-Wire Notes Line
 	10200 5700 7750 5700
 Wire Notes Line
@@
 NoConn ~ 8500 4900
 Wire Wire Line
-	8300 3500 8500 3500
-Wire Wire Line
-	8500 3300 8300 3300
+	8300 3900 8500 3900
+Wire Wire Line
+	8500 3500 8300 3500
 NoConn ~ 8500 3200
+NoConn ~ 8500 3300
+NoConn ~ 8500 4400
+NoConn ~ 8500 4500
+Wire Notes Line
+	10200 2800 10200 5700
 $EndSCHEMATC
